Commit message: add ros2_academy_ws

File: ros2_academy_ws/src/academy_robot_description/robots/academy_robot/academy_robot_plus.urdf.xacro (robot description, xacro)
@@ -81,3 +81,10 @@
     </xacro:unless>
   </xacro:unless>
+  <xacro:arg name="use_fake_hardware" default="true" />
+    <xacro:arg name="com_port" default="/dev/ttyUSB0" />
+    <!-- Import macros -->
+  <xacro:include filename="$(find academy_robot_description)/urdf/robotiq_gripper_macro.xacro" />
+  <xacro:robotiq_gripper name="RobotiqGripperHardwareInterface" prefix="" parent="robot_arm_wrist_3_link" use_fake_hardware="$(arg use_fake_hardware)" com_port="$(arg com_port)" sim_gazebo="$(arg gazebo_ignition)">
+      <origin xyz="0 0 0" rpy="0 0 0" />
+  </xacro:robotiq_gripper>
 </robot>

Commit message: Added gripper_command package, split arm and gripper controllers, updated launch and xacros

File: ros2_academy_ws/src/academy_robot_description/robots/academy_robot/academy_robot_plus.urdf.xacro (robot description, xacro)
@@ -82,5 +82,5 @@
   </xacro:unless>
   <xacro:arg name="use_fake_hardware" default="true" />
-    <xacro:arg name="com_port" default="/dev/ttyUSB0" />
+  <xacro:arg name="com_port" default="/dev/ttyUSB0" />
     <!-- Import macros -->
   <xacro:include filename="$(find academy_robot_description)/urdf/robotiq_gripper_macro.xacro" />

File: ros2_academy_ws/src/academy_robot_description/urdf/robotiq_gripper.ros2_control.xacro (robot description, xacro)
@@ -49,42 +49,32 @@
             <joint name="${prefix}robotiq_85_left_knuckle_joint">
                 <command_interface name="position" />
-                <state_interface name="position">
-                    <param name="initial_value">${gripper_closed_position}</param>
-                </state_interface>
+                <state_interface name="position"/>
                 <state_interface name="velocity"/>
             </joint>
-            <!-- When simulating we need to include the rest of the gripper joints -->
-            <xacro:if value="${use_fake_hardware or sim_isaac or sim_gazebo}">
                 <joint name="${prefix}robotiq_85_right_knuckle_joint">
-                    <xacro:unless value="${sim_gazebo}">
-                        <state_interface name="position"/>
-                        <state_interface name="velocity"/>
-                    </xacro:unless>
+                    <command_interface name="position" />
+                    <state_interface name="position"/>
+                    <state_interface name="velocity"/>
                 </joint>
                 <joint name="${prefix}robotiq_85_left_inner_knuckle_joint">
-                    <xacro:unless value="${sim_gazebo}">
-                        <state_interface name="position"/>
-                        <state_interface name="velocity"/>
-                    </xacro:unless>
+                    <command_interface name="position" />
+                    <state_interface name="position"/>
+                    <state_interface name="velocity"/>
                 </joint>
                 <joint name="${prefix}robotiq_85_right_inner_knuckle_joint">
-                    <xacro:unless value="${sim_gazebo}">
-                        <state_interface name="position"/>
-                        <state_interface name="velocity"/>
-                    </xacro:unless>
+                    <command_interface name="position" />
+                    <state_interface name="position"/>
+                    <state_interface name="velocity"/>
                 </joint>
                 <joint name="${prefix}robotiq_85_left_finger_tip_joint">
-                    <xacro:unless value="${sim_gazebo}">
-                        <state_interface name="position"/>
-                        <state_interface name="velocity"/>
-                    </xacro:unless>
+                    <command_interface name="position" />
+                    <state_interface name="position"/>
+                    <state_interface name="velocity"/>
                 </joint>
                 <joint name="${prefix}robotiq_85_right_finger_tip_joint">
-                    <xacro:unless value="${sim_gazebo}">
-                        <state_interface name="position"/>
-                        <state_interface name="velocity"/>
-                    </xacro:unless>
+                    <command_interface name="position" />
+                    <state_interface name="position"/>
+                    <state_interface name="velocity"/>
                 </joint>
-            </xacro:if>
             <!-- Only add this with fake hardware mode -->
             <xacro:unless value="${sim_gazebo or sim_isaac}">

File: ros2_academy_ws/src/academy_robot_description/urdf/robotiq_gripper_macro.xacro (robot description, xacro)
@@ -245,5 +245,4 @@
             <origin xyz="-0.03060114 0.0 0.05490452" rpy="0 0 0" />
             <limit lower="-0.8" upper="0.0" velocity="0.5" effort="50" />
-            <mimic joint="${prefix}robotiq_85_left_knuckle_joint" multiplier="-1" />
         </joint>
         <joint name="${prefix}robotiq_85_left_finger_joint" type="fixed">
@@ -262,5 +261,5 @@
             <axis xyz="0 -1 0" />
             <origin xyz="0.0127 0.0 0.06142" rpy="0 0 0" />
-            <mimic joint="${prefix}robotiq_85_left_knuckle_joint" />
+            <limit lower="0.0" upper="0.8" velocity="0.5" effort="50" />
         </joint>
         <joint name="${prefix}robotiq_85_right_inner_knuckle_joint" type="continuous">
@@ -269,5 +268,5 @@
             <axis xyz="0 -1 0" />
             <origin xyz="-0.0127 0.0 0.06142" rpy="0 0 0" />
-            <mimic joint="${prefix}robotiq_85_left_knuckle_joint" multiplier="-1" />
+            <limit lower="-0.8" upper="0.0" velocity="0.5" effort="50" />
         </joint>
         <joint name="${prefix}robotiq_85_left_finger_tip_joint" type="continuous">
@@ -276,5 +275,5 @@
             <axis xyz="0 -1 0" />
             <origin xyz="0.00563134 0.0 0.04718515" rpy="0 0 0" />
-            <mimic joint="${prefix}robotiq_85_left_knuckle_joint" multiplier="-1" />
+            <limit lower="-0.8" upper="0.0" velocity="0.5" effort="50" />
         </joint>
         <joint name="${prefix}robotiq_85_right_finger_tip_joint" type="continuous">
@@ -283,5 +282,5 @@
             <axis xyz="0 -1 0" />
             <origin xyz="-0.00563134 0.0 0.04718515" rpy="0 0 0" />
-            <mimic joint="${prefix}robotiq_85_left_knuckle_joint" />
+            <limit lower="0.0" upper="0.8" velocity="0.5" effort="50" />
         </joint>
     </xacro:macro>
