Commit message: Add TCP transform

File: ros2_academy_ws/src/academy_robot_description/urdf/robotiq_gripper_macro.xacro (robot description, xacro)
@@ -270,4 +270,11 @@
             <limit lower="-0.8" upper="0.0" velocity="0.5" effort="50" />
         </joint>
+        <!-- Tool Center Point (TCP) link and joint -->
+        <link name="${prefix}robotiq_85_tcp"/>
+        <joint name="${prefix}robotiq_85_base_link-robotiq_85_tcp" type="fixed">
+            <parent link="${prefix}robotiq_85_base_link" />
+            <child link="${prefix}robotiq_85_tcp"/>
+            <origin xyz="0.0 2.274e-05 0.11" rpy="0 0 0" />
+        </joint>
         <joint name="${prefix}robotiq_85_left_finger_tip_joint" type="continuous">
             <parent link="${prefix}robotiq_85_left_finger_link" />
