Commit message: add collision for top layer

File: ros2_academy_ws/src/academy_robot_description/urdf/bodies/academy_robot/academy_robot_plus_body.urdf.xacro (robot description, xacro)
@@ -56,4 +56,10 @@
         </material>
       </visual>
+      <collision>
+        <origin xyz="0 0 0" rpy="0 0 0" />
+        <geometry>
+          <mesh filename="package://academy_robot_description/meshes/bases/academy_robot/academy_robot_top_cover.stl" />
+        </geometry>
+      </collision>
     </link>
     <joint name="${prefix}top_cover_joint" type="fixed">
