Commit message: added moveit config for ur and gripper

File: ros2_academy_ws/src/Universal_Robots_ROS2_Description/urdf/ur.ros2_control.xacro (robot description, xacro)
@@ -3,5 +3,5 @@
   <xacro:macro name="ur_ros2_control" params="
     name
-    use_fake_hardware:=false fake_sensor_commands:=false
+    use_fake_hardware:=true fake_sensor_commands:=false
     sim_gazebo:=false
     sim_ignition:=false
@@ -37,5 +37,6 @@
         </xacro:if>
         <xacro:unless value="${use_fake_hardware or sim_gazebo or sim_ignition}">
-          <plugin>ur_robot_driver/URPositionHardwareInterface</plugin>
+          <!-- <plugin>ur_robot_driver/URPositionHardwareInterface</plugin> -->
+           <plugin>fake_components/GenericSystem</plugin>
           <param name="robot_ip">${robot_ip}</param>
           <param name="script_filename">${script_filename}</param>

File: ros2_academy_ws/src/academy_robot_description/robots/academy_robot/academy_robot_plus.urdf.xacro (robot description, xacro)
@@ -1,90 +1,4 @@
-<?xml version="1.0"?>
 <robot name="academy_robot" xmlns:xacro="http://wiki.ros.org/xacro">
-  <!-- ***************** -->
-  <!-- Imported elements -->
-  <!-- ***************** -->
-  <!-- Import all posible elements defined in the urdf.xacro files. All these elements are defined as macro:xacros -->
-  <xacro:include filename="$(find academy_robot_description)/urdf/bases/academy_robot/academy_robot_base.urdf.xacro" />
-  <xacro:include filename="$(find academy_robot_description)/urdf/base_hw/academy_robot.ros2_control.urdf" />
-  <xacro:include
-    filename="$(find academy_robot_description)/simulators/gazebo_classic/academy_robot/academy_robot_control.urdf.xacro" />
-  <xacro:include
-    filename="$(find academy_robot_description)/simulators/gazebo_ignition/academy_robot/academy_robot_control.urdf.xacro" />
-  <xacro:include filename="$(find academy_robot_sensors)/urdf/all_sensors.urdf.xacro" />
-  <xacro:include filename="$(find ur_description)/urdf/ur_macro.xacro" />
-  <!-- Properties and Arguments -->
-  <xacro:arg name="namespace" default="robot" />
-  <xacro:arg name="prefix" default="robot_" />
-  <xacro:arg name="gazebo_classic" default="false" />
-  <xacro:arg name="gazebo_ignition" default="false" />
-  <xacro:arg name="ur_type" default="ur5e" />
-  <xacro:arg name="joint_limit_params" default="$(find ur_description)/config/$(arg ur_type)/joint_limits.yaml" />
-  <xacro:arg name="kinematics_params" default="$(find ur_description)/config/$(arg ur_type)/default_kinematics.yaml" />
-  <xacro:arg name="physical_params" default="$(find ur_description)/config/$(arg ur_type)/physical_parameters.yaml" />
-  <xacro:arg name="visual_params" default="$(find ur_description)/config/$(arg ur_type)/visual_parameters.yaml" />
-  <xacro:property name="front_laser_offset_x" value="0.2865" />
-  <xacro:property name="front_laser_offset_y" value="-0.20894" />
-  <xacro:property name="front_laser_offset_z" value="0.2973" />
-  <xacro:property name="rear_laser_offset_x" value="-0.2865" />
-  <xacro:property name="rear_laser_offset_y" value="0.20894" />
-  <xacro:property name="rear_laser_offset_z" value="0.2973" />
-  <xacro:property name="imu_offset_x" value="0.127" />
-  <xacro:property name="imu_offset_y" value="-0.129" />
-  <xacro:property name="imu_offset_z" value="0.212" />
-  <xacro:property name="front_rgbd_camera_offset_x" value="0.35850" />
-  <xacro:property name="front_rgbd_camera_offset_y" value="0.0" />
-  <xacro:property name="front_rgbd_camera_offset_z" value="0.25062" />
-  <!-- Kairos -->
-  <xacro:academy_robot prefix="$(arg prefix)" gazebo_classic="$(arg gazebo_classic)" gazebo_ignition="$(arg gazebo_ignition)" />
-  <!-- Import UR arm -->
-  <!-- Import UR arm -->
-  <xacro:ur_robot tf_prefix="$(arg prefix)arm_" name="$(arg ur_type)" parent="$(arg prefix)top_cover"
-    joint_limits_parameters_file="$(arg joint_limit_params)" kinematics_parameters_file="$(arg kinematics_params)"
-    physical_parameters_file="$(arg physical_params)" visual_parameters_file="$(arg visual_params)"
-    sim_gazebo="$(arg gazebo_classic)" sim_ignition="$(arg gazebo_ignition)">
-    <origin xyz="0 0 0" rpy="0 0 0" />
-  </xacro:ur_robot>
-  <!-- PENDIENTE DE ACTUALIZAR Academy Robot_SENSORS -->
-  <!-- IMU -->
-  <xacro:sensor_vectornav frame_prefix="$(arg prefix)vectornav_" parent="$(arg prefix)base_link" node_namespace="$(arg namespace)"
-    gazebo_classic="$(arg gazebo_classic)" gazebo_ignition="$(arg gazebo_ignition)">
-    <origin xyz="${imu_offset_x} ${imu_offset_y} ${imu_offset_z}" rpy="0 0 0" />
-  </xacro:sensor_vectornav>
-  <!-- SENSORS -->
-  <xacro:sensor_sick_s300 frame_prefix="$(arg prefix)front_laser_" parent="$(arg prefix)base_link"
-    node_namespace="$(arg namespace)" node_name="front_laser" gazebo_classic="$(arg gazebo_classic)"
-    gazebo_ignition="$(arg gazebo_ignition)">
-    <origin xyz="${front_laser_offset_x} ${front_laser_offset_y} ${front_laser_offset_z}" rpy="0 ${-PI} ${3/4*PI}" />
-  </xacro:sensor_sick_s300>
-  <xacro:sensor_sick_s300 frame_prefix="$(arg prefix)rear_laser_" parent="$(arg prefix)base_link"
-    node_namespace="$(arg namespace)" node_name="rear_laser" gazebo_classic="$(arg gazebo_classic)"
-    gazebo_ignition="$(arg gazebo_ignition)">
-    <origin xyz="${rear_laser_offset_x} ${rear_laser_offset_y} ${rear_laser_offset_z}" rpy="0 ${-PI} ${-1/4*PI}" />
-  </xacro:sensor_sick_s300>
-  <!-- CAMERA -->
-  <xacro:sensor_intel_realsense_d435 frame_prefix="$(arg prefix)front_rgbd_camera_" parent="$(arg prefix)base_link"
-    node_namespace="$(arg namespace)" node_name="front_camera" gazebo_classic="$(arg gazebo_classic)"
-    gazebo_ignition="$(arg gazebo_ignition)">
-    <origin xyz="${front_rgbd_camera_offset_x} ${front_rgbd_camera_offset_y} ${front_rgbd_camera_offset_z}" rpy="0 0 0" />
-  </xacro:sensor_intel_realsense_d435>
-  <!-- Controllers -->
-  <xacro:if value="$(arg gazebo_classic)">
-    <xacro:academy_robot_gz_classic_control namespace="$(arg namespace)" prefix="$(arg prefix)" />
-    <xacro:ros_planar_move_gazebo_classic />
-  </xacro:if>
-  <xacro:if value="$(arg gazebo_ignition)">
-    <xacro:academy_robot_gz_ignition_control namespace="$(arg namespace)" prefix="$(arg prefix)" />
-  </xacro:if>
-  <xacro:unless value="$(arg gazebo_classic)">
-    <xacro:unless value="$(arg gazebo_ignition)">
-      <xacro:academy_robot_base_hw_controller />
-    </xacro:unless>
-  </xacro:unless>
-  <xacro:arg name="use_fake_hardware" default="true" />
-  <xacro:arg name="com_port" default="/dev/ttyUSB0" />
-    <!-- Import macros -->
-  <xacro:include filename="$(find academy_robot_description)/urdf/robotiq_gripper_macro.xacro" />
-  <xacro:robotiq_gripper name="RobotiqGripperHardwareInterface" prefix="" parent="robot_arm_wrist_3_link" use_fake_hardware="$(arg use_fake_hardware)" com_port="$(arg com_port)" sim_gazebo="$(arg gazebo_ignition)">
-      <origin xyz="0 0 0" rpy="0 0 0" />
-  </xacro:robotiq_gripper>
+  <xacro:include filename="$(find academy_robot_description)/urdf/academy_robot_base.urdf.xacro" />
+  <xacro:include filename="$(find academy_robot_description)/urdf/ur_gripper.urdf.xacro" />
 </robot>

File: ros2_academy_ws/src/academy_robot_description/urdf/robotiq_gripper.ros2_control.xacro (robot description, xacro)
@@ -8,5 +8,5 @@
         isaac_joint_commands:=/isaac_joint_commands
         isaac_joint_states:=/isaac_joint_states
-        use_fake_hardware:=false
+        use_fake_hardware:=true
         mock_sensor_commands:=false
         com_port:=/dev/ttyUSB0

File: ros2_academy_ws/src/academy_robot_description/urdf/robotiq_gripper_macro.xacro (robot description, xacro)
@@ -10,5 +10,5 @@
         isaac_joint_commands:=/isaac_joint_commands
         isaac_joint_states:=/isaac_joint_states
-        use_fake_hardware:=false
+        use_fake_hardware:=true
         mock_sensor_commands:=false
         include_ros2_control:=true
